File: power.sch (EAGLE design)
At the start: 65 parts, among them J1 POWER_JACKPTH_BREAD, T1 SINGLE_NCHAN_FET, T2 SINGLE_NCHAN_FET, T3 SINGLE_NCHAN_FET, U1 MOSFET_PCHAN_20A, U14 MOSFET_PCHAN_20A, U2 MOSFET_PCHAN_20A

Commit message: Added breakout for USB and charging
Connections:
- net VSOLAR: now also U$1.P3, U$1.P6, U$2.P3, U$2.P6, U$3.P3, U$3.P6, U$4.P3, U$4.P6, U$6.P3, U$6.P6
Changed lines of the file:
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@@
 </segment>
 <segment>
-<wire x1="-99.06" y1="93.98" x2="-93.98" y2="93.98" width="0.1524" layer="91"/>
 <label x="-93.98" y="93.98" size="1.778" layer="95"/>
+<pinref part="U$6" gate="G$1" pin="P6"/>
+<wire x1="-93.98" y1="93.98" x2="-99.06" y2="93.98" width="0.1524" layer="91"/>
 </segment>
 <segment>
-<wire x1="-124.46" y1="93.98" x2="-129.54" y2="93.98" width="0.1524" layer="91"/>
 <label x="-129.54" y="93.98" size="1.778" layer="95" rot="MR0"/>
+<pinref part="U$6" gate="G$1" pin="P3"/>
+<wire x1="-129.54" y1="93.98" x2="-124.46" y2="93.98" width="0.1524" layer="91"/>
 </segment>
 <segment>
-<wire x1="-99.06" y1="60.96" x2="-93.98" y2="60.96" width="0.1524" layer="91"/>
 <label x="-93.98" y="60.96" size="1.778" layer="95"/>
+<pinref part="U$3" gate="G$1" pin="P6"/>
+<wire x1="-93.98" y1="60.96" x2="-99.06" y2="60.96" width="0.1524" layer="91"/>
 </segment>
 <segment>
-<wire x1="-99.06" y1="27.94" x2="-93.98" y2="27.94" width="0.1524" layer="91"/>
 <label x="-93.98" y="27.94" size="1.778" layer="95"/>
+<pinref part="U$1" gate="G$1" pin="P6"/>
+<wire x1="-93.98" y1="27.94" x2="-99.06" y2="27.94" width="0.1524" layer="91"/>
 </segment>
 <segment>
-<wire x1="-99.06" y1="-5.08" x2="-93.98" y2="-5.08" width="0.1524" layer="91"/>
 <label x="-93.98" y="-5.08" size="1.778" layer="95"/>
+<pinref part="U$2" gate="G$1" pin="P6"/>
+<wire x1="-93.98" y1="-5.08" x2="-99.06" y2="-5.08" width="0.1524" layer="91"/>
 </segment>
 <segment>
-<wire x1="-99.06" y1="-38.1" x2="-93.98" y2="-38.1" width="0.1524" layer="91"/>
 <label x="-93.98" y="-38.1" size="1.778" layer="95"/>
+<pinref part="U$4" gate="G$1" pin="P6"/>
+<wire x1="-93.98" y1="-38.1" x2="-99.06" y2="-38.1" width="0.1524" layer="91"/>
 </segment>
 <segment>
-<wire x1="-124.46" y1="-38.1" x2="-129.54" y2="-38.1" width="0.1524" layer="91"/>
 <label x="-129.54" y="-38.1" size="1.778" layer="95" rot="MR0"/>
+<pinref part="U$4" gate="G$1" pin="P3"/>
+<wire x1="-129.54" y1="-38.1" x2="-124.46" y2="-38.1" width="0.1524" layer="91"/>
 </segment>
 <segment>
-<wire x1="-124.46" y1="-5.08" x2="-129.54" y2="-5.08" width="0.1524" layer="91"/>
 <label x="-129.54" y="-5.08" size="1.778" layer="95" rot="MR0"/>
+<pinref part="U$2" gate="G$1" pin="P3"/>
+<wire x1="-129.54" y1="-5.08" x2="-124.46" y2="-5.08" width="0.1524" layer="91"/>
 </segment>
 <segment>
-<wire x1="-124.46" y1="27.94" x2="-129.54" y2="27.94" width="0.1524" layer="91"/>
 <label x="-129.54" y="27.94" size="1.778" layer="95" rot="MR0"/>
+<pinref part="U$1" gate="G$1" pin="P3"/>
+<wire x1="-129.54" y1="27.94" x2="-124.46" y2="27.94" width="0.1524" layer="91"/>
 </segment>
 <segment>
-<wire x1="-124.46" y1="60.96" x2="-129.54" y2="60.96" width="0.1524" layer="91"/>
 <label x="-129.54" y="60.96" size="1.778" layer="95" rot="MR0"/>
+<pinref part="U$3" gate="G$1" pin="P3"/>
+<wire x1="-129.54" y1="60.96" x2="-124.46" y2="60.96" width="0.1524" layer="91"/>
 </segment>
 </net>
