File: mainboard.sch (EAGLE design)
At the start: 91 parts, among them Q3 MOSFET-PCHANNEL, Q4 MOSFET-PCHANNEL, T1 SINGLE_NCHAN_FET, T2 MOSFET_PCHAN_20A, T3 SINGLE_NCHAN_FET, T4 MOSFET_PCHAN_20A, T5 SINGLE_NCHAN_FET, T6 MOSFET_PCHAN_20A, U1 LT3688, U2 TEENSY_3.0+4, U3 RFM23BP, U4 HMC5883LSMD, U5 ITG-3200, U9 MIC803, X1 CRYSTAL.ABS07

Commit message: More main board layout
Parts:
- removed R4: 0R, SparkFun-Resistors:RESISTOR2512
Connections:
- net BATT_INPUT: no longer R1.1
- net N$4: now also R1.1; no longer R1.2, R4.1
- net VBATT: now also R1.2, R20.2, R25.2, ST4.1
- net VREG_IN: no longer R20.2, R25.2, R4.2, ST4.1
Other:
- note added: "Option for 1 or 2 footswitches"
- note removed: "Option for 0, 1, or 2 footswitches"
- moved on the sheet: R1
Changed lines of the file:
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@@
 <part name="ST4" library="SparkFun-Connectors" deviceset="M02" device="3.5MM_LOCK" value="M023.5MM_LOCK"/>
 <part name="R1" library="SparkFun-Resistors" deviceset="RESISTOR" device="2512" value="0R"/>
-<part name="R4" library="SparkFun-Resistors" deviceset="RESISTOR" device="2512" value="0R"/>
 <part name="U$14" library="phonesat" deviceset="CURRENT_MAX4372" device=""/>
 <part name="R5" library="SparkFun-Resistors" deviceset="RESISTOR" device="0805-RES" value=".2R prec"/>
@@
 <wire x1="-180.34" y1="60.96" x2="-190.5" y2="60.96" width="0.1524" layer="91"/>
 <junction x="-180.34" y="60.96"/>
-</segment>
-<segment>
-<pinref part="R20" gate="G$1" pin="2"/>
-<pinref part="R25" gate="G$1" pin="2"/>
-<wire x1="22.86" y1="25.4" x2="22.86" y2="30.48" width="0.1524" layer="91"/>
-<wire x1="22.86" y1="30.48" x2="22.86" y2="35.56" width="0.1524" layer="91"/>
-<wire x1="22.86" y1="30.48" x2="7.62" y2="30.48" width="0.1524" layer="91"/>
-<label x="7.62" y="30.48" size="1.778" layer="95"/>
-<junction x="22.86" y="30.48"/>
+<label x="-175.26" y="38.1" size="1.778" layer="95"/>
 </segment>
 </net>
@@
 <label x="-81.28" y="60.96" size="1.778" layer="95"/>
 </segment>
+<segment>
+<pinref part="R20" gate="G$1" pin="2"/>
+<pinref part="R25" gate="G$1" pin="2"/>
+<wire x1="22.86" y1="25.4" x2="22.86" y2="30.48" width="0.1524" layer="91"/>
+<wire x1="22.86" y1="30.48" x2="22.86" y2="35.56" width="0.1524" layer="91"/>
+<wire x1="22.86" y1="30.48" x2="7.62" y2="30.48" width="0.1524" layer="91"/>
+<label x="7.62" y="30.48" size="1.778" layer="95"/>
+<junction x="22.86" y="30.48"/>
+</segment>
 </net>
 <net name="VBURN_IN" class="0">
@@
 <plain>
 <text x="25.4" y="101.6" size="1.778" layer="97">Footswitch Connections</text>
-<text x="20.32" y="96.52" size="1.778" layer="97">Option for 0, 1, or 2 footswitches</text>
+<text x="22.86" y="96.52" size="1.778" layer="97">Option for 1 or 2 footswitches</text>
 <text x="-124.46" y="139.7" size="1.778" layer="97">Solar Panel Connectors</text>
 <text x="-40.64" y="106.68" size="1.778" layer="97">Battery Terminals</text>
@@
 <instance part="ST3" gate="G$1" x="20.32" y="73.66" rot="R90"/>
 <instance part="ST4" gate="G$1" x="58.42" y="73.66" rot="R90"/>
-<instance part="R1" gate="G$1" x="25.4" y="91.44"/>
-<instance part="R4" gate="G$1" x="50.8" y="91.44"/>
+<instance part="R1" gate="G$1" x="50.8" y="91.44"/>
 </instances>
 <busses>
@@
 </segment>
 </net>
-<net name="VREG_IN" class="0">
-<segment>
-<pinref part="ST4" gate="G$1" pin="1"/>
-<wire x1="58.42" y1="81.28" x2="58.42" y2="91.44" width="0.1524" layer="91"/>
-<wire x1="58.42" y1="91.44" x2="73.66" y2="91.44" width="0.1524" layer="91"/>
-<pinref part="R4" gate="G$1" pin="2"/>
-<wire x1="55.88" y1="91.44" x2="58.42" y2="91.44" width="0.1524" layer="91"/>
-<junction x="58.42" y="91.44"/>
-<label x="73.66" y="91.44" size="1.778" layer="95"/>
-</segment>
-</net>
 <net name="VBURN3" class="0">
 <segment>
@@
 <wire x1="20.32" y1="81.28" x2="20.32" y2="86.36" width="0.1524" layer="91"/>
 <pinref part="ST4" gate="G$1" pin="2"/>
-<wire x1="20.32" y1="86.36" x2="30.48" y2="86.36" width="0.1524" layer="91"/>
-<wire x1="30.48" y1="86.36" x2="45.72" y2="86.36" width="0.1524" layer="91"/>
+<wire x1="20.32" y1="86.36" x2="45.72" y2="86.36" width="0.1524" layer="91"/>
 <wire x1="45.72" y1="86.36" x2="55.88" y2="86.36" width="0.1524" layer="91"/>
 <wire x1="55.88" y1="86.36" x2="55.88" y2="81.28" width="0.1524" layer="91"/>
-<pinref part="R1" gate="G$1" pin="2"/>
-<wire x1="30.48" y1="91.44" x2="30.48" y2="86.36" width="0.1524" layer="91"/>
-<pinref part="R4" gate="G$1" pin="1"/>
+<pinref part="R1" gate="G$1" pin="1"/>
 <wire x1="45.72" y1="91.44" x2="45.72" y2="86.36" width="0.1524" layer="91"/>
-<junction x="30.48" y="86.36"/>
 <junction x="45.72" y="86.36"/>
 </segment>
@@
 <wire x1="17.78" y1="81.28" x2="17.78" y2="91.44" width="0.1524" layer="91"/>
 <wire x1="17.78" y1="91.44" x2="2.54" y2="91.44" width="0.1524" layer="91"/>
-<pinref part="R1" gate="G$1" pin="1"/>
-<wire x1="17.78" y1="91.44" x2="20.32" y2="91.44" width="0.1524" layer="91"/>
-<junction x="17.78" y="91.44"/>
 <wire x1="-27.94" y1="99.06" x2="2.54" y2="99.06" width="0.1524" layer="91"/>
 <wire x1="2.54" y1="99.06" x2="2.54" y2="91.44" width="0.1524" layer="91"/>
@@
 </segment>
 </net>
+<net name="VBATT" class="0">
+<segment>
+<pinref part="ST4" gate="G$1" pin="1"/>
+<wire x1="58.42" y1="81.28" x2="58.42" y2="91.44" width="0.1524" layer="91"/>
+<wire x1="58.42" y1="91.44" x2="73.66" y2="91.44" width="0.1524" layer="91"/>
+<pinref part="R1" gate="G$1" pin="2"/>
+<wire x1="55.88" y1="91.44" x2="58.42" y2="91.44" width="0.1524" layer="91"/>
+<junction x="58.42" y="91.44"/>
+<label x="73.66" y="91.44" size="1.778" layer="95"/>
+</segment>
+</net>

Commit message: main board layout work
Parts:
- added JP1: (no value), SparkFun-Connectors:M041.27MM
- R5, R8: value .2R prec -> .1R prec
Connections:
- net I_BATT: now also U2.14/A0; no longer U2.15/A1
- net N$37: now also U2.15/A1; no longer U2.14/A0
Other:
- moved on the sheet: R22, R24, ST5
Changed lines of the file:
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@@
 <part name="R1" library="SparkFun-Resistors" deviceset="RESISTOR" device="2512" value="0R"/>
 <part name="U$14" library="phonesat" deviceset="CURRENT_MAX4372" device=""/>
-<part name="R5" library="SparkFun-Resistors" deviceset="RESISTOR" device="0805-RES" value=".2R prec"/>
+<part name="R5" library="SparkFun-Resistors" deviceset="RESISTOR" device="0805-RES" value=".1R prec"/>
 <part name="C12" library="SparkFun-Capacitors" deviceset="CAP" device="0805" value=".1uF"/>
 <part name="GND20" library="SparkFun" deviceset="GND" device=""/>
@@
 <part name="GND21" library="SparkFun" deviceset="GND" device=""/>
 <part name="P+2" library="SparkFun" deviceset="3.3V" device=""/>
-<part name="R8" library="SparkFun-Resistors" deviceset="RESISTOR" device="0805-RES" value=".2R prec"/>
+<part name="R8" library="SparkFun-Resistors" deviceset="RESISTOR" device="0805-RES" value=".1R prec"/>
 <part name="U3" library="RFM23BP" deviceset="RFM23BP" device=""/>
 <part name="U5" library="SparkFun-Sensors" deviceset="ITG-3200" device=""/>
@@
 <part name="C23" library="SparkFun-Capacitors" deviceset="CAP" device="0805" value="0.1uF"/>
 <part name="GND14" library="SparkFun" deviceset="GND" device=""/>
+<part name="JP1" library="SparkFun-Connectors" deviceset="M04" device="1.27MM"/>
 </parts>
 <sheets>
@@
 <instance part="P+4" gate="G$1" x="93.98" y="-5.08"/>
 <instance part="P+6" gate="G$1" x="104.14" y="-5.08"/>
-<instance part="R22" gate="G$1" x="134.62" y="-25.4" rot="R90"/>
-<instance part="R24" gate="G$1" x="134.62" y="-40.64" rot="R90"/>
-<instance part="GND28" gate="1" x="134.62" y="-50.8"/>
+<instance part="R22" gate="G$1" x="134.62" y="-22.86" rot="R90"/>
+<instance part="R24" gate="G$1" x="134.62" y="-38.1" rot="R90"/>
+<instance part="GND28" gate="1" x="134.62" y="-48.26"/>
 <instance part="P+8" gate="G$1" x="210.82" y="7.62"/>
 <instance part="GND29" gate="1" x="210.82" y="-22.86"/>
@@
 <segment>
 <pinref part="R24" gate="G$1" pin="1"/>
-<wire x1="134.62" y1="-45.72" x2="134.62" y2="-48.26" width="0.1524" layer="91"/>
+<wire x1="134.62" y1="-43.18" x2="134.62" y2="-45.72" width="0.1524" layer="91"/>
 <pinref part="GND28" gate="1" pin="GND"/>
 </segment>
@@
 <pinref part="R22" gate="G$1" pin="1"/>
 <pinref part="R24" gate="G$1" pin="2"/>
+<wire x1="134.62" y1="-27.94" x2="134.62" y2="-30.48" width="0.1524" layer="91"/>
+<pinref part="U2" gate="G$1" pin="15/A1"/>
 <wire x1="134.62" y1="-30.48" x2="134.62" y2="-33.02" width="0.1524" layer="91"/>
-<pinref part="U2" gate="G$1" pin="14/A0"/>
-<wire x1="134.62" y1="-33.02" x2="134.62" y2="-35.56" width="0.1524" layer="91"/>
-<wire x1="81.28" y1="-33.02" x2="134.62" y2="-33.02" width="0.1524" layer="91"/>
-<junction x="134.62" y="-33.02"/>
+<wire x1="81.28" y1="-30.48" x2="134.62" y2="-30.48" width="0.1524" layer="91"/>
+<junction x="134.62" y="-30.48"/>
 </segment>
 </net>
@@
 <segment>
 <pinref part="R22" gate="G$1" pin="2"/>
-<wire x1="134.62" y1="-20.32" x2="134.62" y2="-10.16" width="0.1524" layer="91"/>
-<label x="134.62" y="-10.16" size="1.778" layer="95" rot="MR270"/>
-</segment>
-</net>
-<net name="I_BATT" class="0">
-<segment>
-<pinref part="U2" gate="G$1" pin="15/A1"/>
-<wire x1="81.28" y1="-30.48" x2="121.92" y2="-30.48" width="0.1524" layer="91"/>
-<label x="121.92" y="-30.48" size="1.778" layer="95" rot="MR0"/>
+<wire x1="134.62" y1="-17.78" x2="134.62" y2="-7.62" width="0.1524" layer="91"/>
+<label x="134.62" y="-7.62" size="1.778" layer="95" rot="MR270"/>
 </segment>
 </net>
@@
 <wire x1="50.8" y1="-10.16" x2="25.4" y2="-10.16" width="0.1524" layer="91"/>
 <label x="25.4" y="-10.16" size="1.778" layer="95"/>
+</segment>
+</net>
+<net name="I_BATT" class="0">
+<segment>
+<pinref part="U2" gate="G$1" pin="14/A0"/>
+<wire x1="81.28" y1="-33.02" x2="121.92" y2="-33.02" width="0.1524" layer="91"/>
+<label x="121.92" y="-33.02" size="1.778" layer="95" rot="MR0"/>
 </segment>
 </net>
@@
 <text x="-124.46" y="139.7" size="1.778" layer="97">Solar Panel Connectors</text>
 <text x="-40.64" y="106.68" size="1.778" layer="97">Battery Terminals</text>
-<text x="5.08" y="43.18" size="1.778" layer="97">Burn Wire 3 Terminal</text>
+<text x="40.64" y="55.88" size="1.778" layer="97">Burn Wire 3 Terminal</text>
 </plain>
 <instances>
@@
 <instance part="GND4" gate="1" x="-25.4" y="91.44"/>
 <instance part="GND5" gate="1" x="-25.4" y="73.66"/>
-<instance part="ST5" gate="G$1" x="7.62" y="33.02"/>
-<instance part="GND6" gate="1" x="17.78" y="27.94"/>
+<instance part="ST5" gate="G$1" x="43.18" y="45.72"/>
+<instance part="GND6" gate="1" x="53.34" y="40.64"/>
 <instance part="GND8" gate="1" x="-111.76" y="109.22"/>
 <instance part="GND9" gate="1" x="-111.76" y="73.66"/>
@@
 <instance part="ST4" gate="G$1" x="58.42" y="73.66" rot="R90"/>
 <instance part="R1" gate="G$1" x="50.8" y="91.44"/>
+<instance part="JP1" gate="G$1" x="-43.18" y="38.1"/>
 </instances>
 <busses>
@@
 <segment>
 <pinref part="ST5" gate="G$1" pin="1"/>
-<wire x1="15.24" y1="33.02" x2="17.78" y2="33.02" width="0.1524" layer="91"/>
-<wire x1="17.78" y1="33.02" x2="17.78" y2="30.48" width="0.1524" layer="91"/>
+<wire x1="50.8" y1="45.72" x2="53.34" y2="45.72" width="0.1524" layer="91"/>
+<wire x1="53.34" y1="45.72" x2="53.34" y2="43.18" width="0.1524" layer="91"/>
 <pinref part="GND6" gate="1" pin="GND"/>
 </segment>
@@
 <segment>
 <pinref part="ST5" gate="G$1" pin="2"/>
-<wire x1="15.24" y1="35.56" x2="22.86" y2="35.56" width="0.1524" layer="91"/>
-<label x="22.86" y="35.56" size="1.778" layer="95"/>
-</segment>
-</net>
+<wire x1="50.8" y1="48.26" x2="58.42" y2="48.26" width="0.1524" layer="91"/>
+<label x="58.42" y="48.26" size="1.778" layer="95"/>
+</segment>
+</net>
