File: mainboard.brd (EAGLE design)
At the start: 90.2 x 95.9 mm, 78 parts, among them J1 POWER_JACKPTH_LOCK, T1 SINGLE_NCHAN_FET, T10 SINGLE_NCHAN_FET, T2 MOSFET_PCHAN_20A, T3 SINGLE_NCHAN_FET, T4 MOSFET_PCHAN_20A, T5 SINGLE_NCHAN_FET, T6 MOSFET_PCHAN_20A, T7 MOSFET_PCHAN_20A, T8 SINGLE_NCHAN_FET, T9 MOSFET_PCHAN_20A, U1 MURATA_REG_OKL-T3-W12, U2 TEENSY_3.0+4, U3 RFM23BP, U4 HMC5883LSMD, U5 ITG-3200, U7 CURRENT_MAX4372, U8 CURRENT_MAX4372

Commit message: Some layout work
Parts:
- moved X1 240.5 mm to (125.2, 37.1), turned to 90 degrees
- moved R14 177.6 mm to (62.9, 17.1), turned to 90 degrees
- moved C3 80.8 mm to (67.9, 27.1), turned to 180 degrees
- moved U$3 77.8 mm to (51.0, 38.0)
- moved U1 70.6 mm to (72.7, 18.0), turned to 0 degrees
- moved R9 62.2 mm to (79.3, 9.90), turned to 0 degrees
- moved C2 57.4 mm to (82.1, 18.0), turned to 0 degrees
- moved C1 56.3 mm to (83.1, 21.5), turned to 0 degrees
- moved JP10 53.2 mm to (119.2, 26.4)
- moved R8 44.7 mm to (69.2, 30.6), turned to 90 degrees
- moved U7 41.5 mm to (72.9, 30.6), turned to 90 degrees
- moved C13 36.5 mm to (75.3, 33.1), turned to 0 degrees
- moved C31 32.6 mm to (100.7, 81.3)
- moved R3 32.6 mm to (104.1, 78.7)
- moved T3 32.6 mm to (100.7, 77.4)
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Connections:
- net N$11: now also S3.3; no longer S3.1
- net N_ENAB_REG: now also U$3.15; no longer U$3.10
Routing:
- net N$13: track 0.00 -> 96.9 mm, vias 0 -> 1
- net N$11: track 0.00 -> 95.2 mm, vias 0 -> 1
- net PGM_RST: track 0.00 -> 51.2 mm
- net PGM_VCC: track 0.00 -> 50.0 mm, vias 0 -> 1
- net I_BATT: track 0.00 -> 46.5 mm, vias 0 -> 1
- net UART1_TX: track 0.00 -> 42.7 mm
- net UART1_RX: track 0.00 -> 42.7 mm
- net N_ENAB_REG: track 0.00 -> 15.7 mm
- net GND: track 44.6 -> 56.7 mm, vias 19 -> 24
- net VREG_IN: track 0.00 -> 8.39 mm
- net 3.3V: track 17.8 -> 24.2 mm, vias 6 -> 7
- net VSOLAR: track 0.00 -> 4.04 mm, vias 0 -> 1
- net VBATT: track 0.00 -> 4.00 mm
- net SPI_SCK: track 32.0 -> 29.9 mm

Commit message: More layout work
Parts:
- moved R10 136.9 mm to (73.1, 52.2), turned to 180 degrees
- moved R27 105.4 mm to (16.2, 61.9)
- moved T1 105.4 mm to (11.8, 61.9)
- moved C30 105.4 mm to (7.99, 61.9)
- moved T2 105.4 mm to (10.6, 57.3)
- moved R28 105.4 mm to (10.5, 65.4)
- moved R4 87.1 mm to (7.20, 66.2)
- moved C31 46.8 mm to (67.9, 47.9), turned to 270 degrees
- moved R3 43.4 mm to (70.5, 51.3), turned to 270 degrees
- moved T3 41.3 mm to (71.8, 47.9), turned to 270 degrees
- moved R2 39.5 mm to (73.2, 44.8), turned to 270 degrees
- moved T4 33.5 mm to (77.3, 47.9), turned to 0 degrees
Routing:
- net ENAB_BURN2: track 0.00 -> 46.6 mm, vias 0 -> 1
- net ENAB_BURN1: track 0.00 -> 36.5 mm
- net VBURN1: track 0.00 -> 15.5 mm
- net VBURN_IN: track 0.00 -> 14.7 mm
- net GND: track 56.7 -> 70.2 mm, vias 24 -> 28
- net VBURN2: track 0.00 -> 10.4 mm
- net N$3: track 0.00 -> 10.3 mm
- net N$24: track 0.00 -> 4.71 mm
- net N$2: track 0.00 -> 4.19 mm
- net N$21: track 0.00 -> 4.17 mm

Commit message: More layout work
Parts:
- moved R17 229.8 mm to (19.2, 83.5)
- moved R16 229.2 mm to (19.2, 81.1), turned to 180 degrees
- moved T10 223.1 mm to (15.4, 79.8), turned to 180 degrees
- moved C5 221.8 mm to (15.4, 83.5), turned to 180 degrees
- moved R15 214.4 mm to (12.2, 78.4), turned to 180 degrees
- moved T9 210.8 mm to (17.3, 72.6), turned to 180 degrees
- moved X1 126.3 mm to (4.30, 73.7), turned to 270 degrees
- moved ST5 64.4 mm to (79.0, 77.4), turned to 90 degrees
- moved ST3 55.6 mm to (71.9, 70.4), turned to 90 degrees
- moved ST1 48.5 mm to (79.0, 70.4), turned to 90 degrees
- moved ST4 45.2 mm to (71.9, 63.4), turned to 90 degrees
- moved ST2 36.0 mm to (79.0, 63.4), turned to 90 degrees
- moved R5 18.9 mm to (99.2, 39.9)
- moved U8 18.9 mm to (99.2, 43.1)
- moved C12 18.9 mm to (97.3, 46.4)
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Routing:
- net N$1: track 0.00 -> 94.1 mm
- net BATT_INPUT: track 0.00 -> 82.6 mm
- net ENAB_GPS: track 0.00 -> 52.9 mm
- net VBATT: track 4.00 -> 46.0 mm
- net UART3_TX: track 0.00 -> 34.7 mm, vias 0 -> 1
- net UART3_RX: track 0.00 -> 32.3 mm, vias 0 -> 1
- net I2C_SCL: track 4.92 -> 34.4 mm, vias 0 -> 2
- net I2C_SDA: track 4.93 -> 34.4 mm, vias 0 -> 2
- net GPS_PWR: track 0.00 -> 14.3 mm
- net GND: track 70.2 -> 80.0 mm, vias 28 -> 31
- net N$12: track 0.00 -> 5.50 mm
- net N$10: track 0.00 -> 4.37 mm
- net N$4: track 0.00 -> 3.14 mm
- net N$44: track 9.31 -> 8.56 mm
- added copper zone on layer 2, net N$14
- added copper zone on layer 15, net N$15
- added copper zone on layer 16, net N$16

Commit message: More layout work
Parts:
- moved JP10 109.7 mm to (10.2, 38.5), turned to 270 degrees
- moved JP9 102.3 mm to (14.0, 8.30)
- moved JP12 95.3 mm to (30.0, 91.8)
- moved SMA1 0.50 mm to (11.3, 21.5)
Routing:
- net N$19: track 7.82 -> 7.32 mm
Other:
- board text added: "+"
- board text added: "-"
- board text added: "Batteries"
- board text added: "Foot Switches"
- board text added: "Rail Switch"
Changed lines of the file:
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@@
 <text x="27.3" y="5.5" size="1.778" layer="21">FLIGHT</text>
 <wire x1="50.585" y1="12.5" x2="50.585" y2="17.5" width="0.4064" layer="21"/>
+<text x="84.4" y="73.6" size="1.778" layer="27" rot="R90">-</text>
+<text x="84.4" y="66.7" size="1.778" layer="27" rot="R90">-</text>
+<text x="83" y="69.4" size="1.778" layer="27">+</text>
+<text x="83" y="62.4" size="1.778" layer="27">+</text>
+<text x="84.5" y="75.8" size="1.016" layer="27" rot="R90">Rail Switch</text>
+<text x="85.8" y="65.8" size="1.016" layer="25" rot="R90">Batteries</text>
+<text x="67.6" y="73.3" size="1.016" layer="26" rot="MR270">Foot Switches</text>
 </plain>
 <attributes>
@@
 <attribute name="NAME" x="71.09" y="90.265" size="0.6096" layer="25"/>
 </element>
-<element name="SMA1" library="con-coax" package="BU-SMA-V" value="BU-SMA-V" x="10.82" y="21.5" smashed="yes" rot="MR180">
-<attribute name="OC_NEWARK" value="unknown" x="-44.53" y="-1.34" size="1.778" layer="28" rot="MR180" display="off"/>
-<attribute name="MPN" value="" x="-44.53" y="-1.34" size="1.778" layer="28" rot="MR180" display="off"/>
-<attribute name="MF" value="" x="-44.53" y="-1.34" size="1.778" layer="28" rot="MR180" display="off"/>
-<attribute name="OC_FARNELL" value="unknown" x="-44.53" y="-1.34" size="1.778" layer="28" rot="MR180" display="off"/>
+<element name="SMA1" library="con-coax" package="BU-SMA-V" value="BU-SMA-V" x="11.32" y="21.5" smashed="yes" rot="MR180">
+<attribute name="OC_NEWARK" value="unknown" x="-44.03" y="-1.34" size="1.778" layer="28" rot="MR180" display="off"/>
+<attribute name="MPN" value="" x="-44.03" y="-1.34" size="1.778" layer="28" rot="MR180" display="off"/>
+<attribute name="MF" value="" x="-44.03" y="-1.34" size="1.778" layer="28" rot="MR180" display="off"/>
+<attribute name="OC_FARNELL" value="unknown" x="-44.03" y="-1.34" size="1.778" layer="28" rot="MR180" display="off"/>
 </element>
 <element name="U2" library="Teensy3.0" package="TEENSY_3.0+4" value="TEENSY_3.0+4" x="45.085" y="77" smashed="yes">
@@
 <element name="JP1" library="SparkFun-Connectors" package="MOLEX-1X3_LOCK" value="" x="3.9" y="50.4825" rot="R270"/>
 <element name="JP8" library="SparkFun-Connectors" package="MOLEX-1X3_LOCK" value="" x="86" y="45.4025" rot="R90"/>
-<element name="JP9" library="SparkFun-Connectors" package="MOLEX-1X3_LOCK" value="" x="102.8" y="59"/>
-<element name="JP10" library="SparkFun-Connectors" package="MOLEX-1X3_LOCK" value="" x="119.2" y="26.4" rot="MR0"/>
+<element name="JP9" library="SparkFun-Connectors" package="MOLEX-1X3_LOCK" value="" x="14" y="8.3"/>
+<element name="JP10" library="SparkFun-Connectors" package="MOLEX-1X3_LOCK" value="" x="10.2" y="38.5" rot="MR270"/>
 <element name="JP11" library="SparkFun-Connectors" package="MOLEX-1X3_LOCK" value="" x="59.3" y="4"/>
-<element name="JP12" library="SparkFun-Connectors" package="MOLEX-1X3_LOCK" value="" x="116.2" y="51.1" rot="R180"/>
-<element name="ST5" library="SparkFun-Connectors" package="SCREWTERMINAL-3.5MM-2_LOCK" value="M023.5MM_LOCK" x="79" y="77.4" rot="R90"/>
+<element name="JP12" library="SparkFun-Connectors" package="MOLEX-1X3_LOCK" value="" x="30" y="91.8" rot="R180"/>
+<element name="ST5" library="SparkFun-Connectors" package="SCREWTERMINAL-3.5MM-2_LOCK" value="M023.5MM_LOCK" x="79.01" y="77.4" smashed="yes" rot="R90"/>
 <element name="T7" library="phonesat" package="SO8" value="MOSFET_PCHAN_20A" x="-54.3" y="-52.2"/>
 <element name="T8" library="phonesat" package="SOT23-3" value="SINGLE_NCHAN_FET" x="-57" y="-58.9"/>
@@
 <wire x1="12.9" y1="83.5" x2="12.7" y2="83.7" width="0.4064" layer="16"/>
 <wire x1="124.47" y1="93.86" x2="124.57" y2="96.37" width="0" layer="19" extent="1-1"/>
-<wire x1="102.8" y1="59.127" x2="124.47" y2="93.86" width="0" layer="19" extent="1-1"/>
-<wire x1="96.45" y1="46.4" x2="102.8" y2="59.127" width="0" layer="19" extent="1-1"/>
+<wire x1="82.55" y1="90.805" x2="124.47" y2="93.86" width="0" layer="19" extent="1-1"/>
+<wire x1="94.9" y1="46.6" x2="85.873" y2="45.4025" width="0" layer="19" extent="16-16"/>
 <wire x1="100.15" y1="44.6301" x2="96.45" y2="46.4" width="0" layer="19" extent="1-1"/>
-<wire x1="85.873" y1="45.4025" x2="94.9" y2="46.6" width="0" layer="19" extent="16-16"/>
 <wire x1="106.81" y1="36.71" x2="101.7" y2="44.4" width="0" layer="19" extent="1-16"/>
-<wire x1="116.2" y1="50.973" x2="102.8" y2="59.127" width="0" layer="19" extent="1-1"/>
-<wire x1="119.2" y1="26.527" x2="106.81" y2="36.71" width="0" layer="19" extent="1-1"/>
 <wire x1="-57.9" y1="1.8" x2="5.09" y2="5.08" width="0" layer="19" extent="1-1"/>
 <wire x1="-49.4" y1="-57.4" x2="-57.9" y2="1.8" width="0" layer="19" extent="1-1"/>
@@
 <wire x1="126.685" y1="82.88" x2="127.955" y2="82.88" width="0" layer="19" extent="1-1"/>
 <wire x1="125.415" y1="82.88" x2="126.685" y2="82.88" width="0" layer="19" extent="1-1"/>
-<wire x1="107.88" y1="59.127" x2="125.415" y2="82.88" width="0" layer="19" extent="1-1"/>
+<wire x1="19.08" y1="8.427" x2="125.415" y2="82.88" width="0" layer="19" extent="1-1"/>
 </signal>
 <signal name="3.3V">
@@
 <via x="96.3" y="41.6" extent="1-16" drill="0.6"/>
 <wire x1="96.3" y1="41.6" x2="96.1" y2="41.4" width="0.6096" layer="15"/>
-<wire x1="113.66" y1="51.227" x2="105.34" y2="58.873" width="0" layer="19" extent="1-1"/>
-<wire x1="98.25" y1="41.6299" x2="113.66" y2="51.227" width="0" layer="19" extent="1-1"/>
 <wire x1="86.127" y1="47.9425" x2="96.1" y2="41.4" width="0" layer="19" extent="1-15"/>
-<wire x1="116.66" y1="26.273" x2="98.28" y2="39.85" width="0" layer="19" extent="1-1"/>
 </signal>
 <signal name="N$4">
@@
 <contactref element="U3" pad="ANT"/>
 <contactref element="SMA1" pad="1"/>
-<wire x1="10.82" y1="21.5" x2="18.58" y2="21.5" width="0.8128" layer="1"/>
+<wire x1="11.32" y1="21.5" x2="18.58" y2="21.5" width="0.8128" layer="1"/>
 <wire x1="18.58" y1="21.5" x2="18.62" y2="21.54" width="0.8128" layer="1"/>
 </signal>
@@
 <wire x1="79.01" y1="67.0678" x2="79.3678" y2="67.0678" width="1.27" layer="16"/>
 <wire x1="79.3678" y1="67.0678" x2="81.9" y2="64.5356" width="1.27" layer="16"/>
-<wire x1="79.01" y1="74.0678" x2="79.01" y2="77.2122" width="1.27" layer="1"/>
-<wire x1="79.01" y1="77.2122" x2="79" y2="77.2222" width="1.27" layer="1"/>
+<wire x1="79.01" y1="74.0678" x2="79.01" y2="77.2222" width="1.27" layer="1"/>
 </signal>
 <signal name="N$8">
