File: antenna.sch (EAGLE design)
At the start: 23 parts, among them X1 BU-SMA-V

Commit message: Fixed solar cell footprints
Parts:
- D1, D2, D3, D4, D5, D6: device phonesat:SB_DIODE -> Solar:SB_DIODE
- SL1, SL10, SL2, SL3, SL4, SL5, SL6, SL7, SL8, SL9: device phonesat:SOLAR_CELL -> Solar:SOLAR_CELL
Changed lines of the file:
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@@
 <part name="U$1" library="TapeAntenna" deviceset="TAPEANTENNA" device=""/>
 <part name="U$2" library="TapeAntenna" deviceset="TAPEANTENNA" device=""/>
-<part name="SL3" library="phonesat" deviceset="SOLAR_CELL" device=""/>
-<part name="D3" library="phonesat" deviceset="SB_DIODE" device=""/>
-<part name="SL4" library="phonesat" deviceset="SOLAR_CELL" device=""/>
-<part name="SL1" library="phonesat" deviceset="SOLAR_CELL" device=""/>
-<part name="SL7" library="phonesat" deviceset="SOLAR_CELL" device=""/>
-<part name="SL8" library="phonesat" deviceset="SOLAR_CELL" device=""/>
-<part name="SL2" library="phonesat" deviceset="SOLAR_CELL" device=""/>
-<part name="D2" library="phonesat" deviceset="SB_DIODE" device=""/>
-<part name="D4" library="phonesat" deviceset="SB_DIODE" device=""/>
-<part name="D5" library="phonesat" deviceset="SB_DIODE" device=""/>
-<part name="D6" library="phonesat" deviceset="SB_DIODE" device=""/>
-<part name="D1" library="phonesat" deviceset="SB_DIODE" device=""/>
+<part name="SL3" library="Solar" deviceset="SOLAR_CELL" device=""/>
+<part name="D3" library="Solar" deviceset="SB_DIODE" device=""/>
+<part name="SL4" library="Solar" deviceset="SOLAR_CELL" device=""/>
+<part name="SL1" library="Solar" deviceset="SOLAR_CELL" device=""/>
+<part name="SL7" library="Solar" deviceset="SOLAR_CELL" device=""/>
+<part name="SL8" library="Solar" deviceset="SOLAR_CELL" device=""/>
+<part name="SL2" library="Solar" deviceset="SOLAR_CELL" device=""/>
+<part name="D2" library="Solar" deviceset="SB_DIODE" device=""/>
+<part name="D4" library="Solar" deviceset="SB_DIODE" device=""/>
+<part name="D5" library="Solar" deviceset="SB_DIODE" device=""/>
+<part name="D6" library="Solar" deviceset="SB_DIODE" device=""/>
+<part name="D1" library="Solar" deviceset="SB_DIODE" device=""/>
 <part name="GND2" library="SparkFun" deviceset="GND" device=""/>
-<part name="SL6" library="phonesat" deviceset="SOLAR_CELL" device=""/>
-<part name="SL5" library="phonesat" deviceset="SOLAR_CELL" device=""/>
-<part name="SL9" library="phonesat" deviceset="SOLAR_CELL" device=""/>
-<part name="SL10" library="phonesat" deviceset="SOLAR_CELL" device=""/>
+<part name="SL6" library="Solar" deviceset="SOLAR_CELL" device=""/>
+<part name="SL5" library="Solar" deviceset="SOLAR_CELL" device=""/>
+<part name="SL9" library="Solar" deviceset="SOLAR_CELL" device=""/>
+<part name="SL10" library="Solar" deviceset="SOLAR_CELL" device=""/>
 <part name="GND3" library="SparkFun" deviceset="GND" device=""/>
 <part name="JP1" library="SparkFun-Connectors" deviceset="M03" device="POLAR_LOCK"/>
