File: Mainboard.sch (EAGLE design)
At the start: 84 parts, among them J1 POWER_JACKPTH_LOCK, T1 MOSFET_PCHAN_20A, T10 SINGLE_NCHAN_FET, T2 SINGLE_NCHAN_FET, T3 MOSFET_PCHAN_20A, T4 SINGLE_NCHAN_FET, T5 MOSFET_PCHAN_20A, T6 SINGLE_NCHAN_FET, T7 MOSFET_PCHAN_20A, T8 SINGLE_NCHAN_FET, T9 MOSFET_PCHAN_20A, U1 RFM23BP, U2 ARDUINO_PRO_MINI, U3 HMC5883LSMD, U4 TEENSY_3.0+4, U5 ITG-3200, U6 CURRENT_MAX4372, U7 MURATA_REG_OKL-T3-W12, U8 CURRENT_MAX4372

Commit message: Added kicksat2 mainboard
Took a snapshot of kicksat1 files, then added new mainboard schematic/layout/libraries
Parts:
- removed S1: DPDT, SparkFun-Electromechanical:SWITCH-DPDTAYZ0202
- removed SMA1: BU-SMA-V, con-coax:BU-SMA-V
- removed ST1, ST2, ST3, ST4, ST5: M023.5MM_LOCK, SparkFun-Connectors:M023.5MM_LOCK
- removed T10, T6, T8: SINGLE_NCHAN_FET, phonesat:SINGLE_NCHAN_FET
- removed T7, T9: MOSFET_PCHAN_20A, phonesat:MOSFET_PCHAN_20A
- added C20, C33: 2.2uF, SparkFun-Capacitors:2.2UF-0603-10V-20%
- added C21: 2.2nF, SparkFun-Capacitors:2.2NF/2200PF-0603-50V-10%
- added C22, C29, C30, C31, C32: .1uF, SparkFun-Capacitors:CAP0603-CAP
- added C23, C27, C28: 0.1uF, SparkFun-Capacitors:0.1UF-0603-25V-5%
- added C24: 3.3nF, SparkFun-Capacitors:3.3NF-0603-100V-10%
- added C25: 1.0uF, SparkFun-Capacitors:1.0UF-0603-16V-10%
- added C26: 22uF, SparkFun-Capacitors:0.1UF-0603-25V-5%
- added C34: 0.33µF, SparkFun-Capacitors:0.33UF/330NF-0805-50V-10%
- added C36: 10uF, SparkFun-Capacitors:10UF-0603-6.3V-20%
- added D1: DFLS130L, BrownSpaceEngineering:DFLS130L
- added D2: GREEN, SparkFun-LED:LED-GREEN0603
- added D3: 200mA/70V, SparkFun-DiscreteSemi:BAV99
- added F1: 1206L200, BrownSpaceEngineering:PTCFUSE1206
- added F2: 500mA, SparkFun-PowerIC:PTCSMD
- added FRAME4: FRAME-LETTER, SparkFun-Aesthetics:FRAME-LETTER
- added IC1: LM234Z, linear:LM234Z
- added J2: POWER_JACKPTH_LOCK, SparkFun-Connectors:POWER_JACKPTH_LOCK
- added JP10, JP13, JP14, JP17, JP9: (no value), SparkFun-Connectors:M03POLAR_LOCK
- added JP11, JP12, JP15, JP16, JP18: M023.5MM_LOCK, SparkFun-Connectors:M023.5MM_LOCK
- added JP19, JP20, JP21: JUMPER-PAD-3-2OF3_NC_BY_TRACE_SMALL, SparkFun-Passives:JUMPER-PAD-3-2OF3_NC_BY_TRACE_SMALL
- added JP22, JP24, JP25, JP26, JP27, JP28: (no value), pinhead:PINHD-1X1
- added L1: FB - 30Ohm, SparkFun-Passives:INDUCTOR0603
- added L3: 3.3uH, BrownSpaceEngineering:IND1812
- added L4: 56uH, BrownSpaceEngineering:IND1812
- added Q1, Q2, Q3, Q4, Q5: IRLML5103, User-Submitted:MOSFET-PCHANNEL
- added R28, R31, R34: 4.7k, SparkFun-Resistors:RESISTOR0603
- added R29, R30, R32, R33: 4, resistor:R-US_R0603
- added R35, R36, R37, R38: 10k, SparkFun-Resistors:RESISTOR0603
- added R39, R40, R41, R42: 3.3k, SparkFun-Resistors:RESISTOR0603
- added R43, R45: 330, SparkFun-Resistors:330OHM1/10W1%(0603)
- added R44, R46, R47, R48, R49, R50, R51, R52, R53, R54, R55: 10K, SparkFun-Resistors:10KOHM-1/10W-1%(0603)0603
- added U10: EP2W+, maholli:EP2W+
- added U11: S1216V8, maholli:S1216V8
- added U12: Value, maholli:ADS124S08IPBSR
- added U9: LC05111C13MTTTG, BrownSpaceEngineering:LC05111C13MTTTG
- added X1, X2, X3: BU-SMA-V, con-coax:BU-SMA-V
- added Y1: 32.768kHz, samd21-temp:CRYSTAL3.2X1.5MM
- C1: value 0.1uF -> 10uF; device SparkFun-Capacitors:CAP0805 -> SparkFun-Capacitors:10UF-6.3V-20%(0603)
- C10, C12: value 22uF -> 0.1uF; device SparkFun-Capacitors:CAP1206 -> SparkFun-Capacitors:0.1UF-25V(+80/-20%)(0603)
- C11, C13, C9: value .1uF -> 0.1uF; device SparkFun-Capacitors:CAP0805 -> SparkFun-Capacitors:0.1UF-25V(+80/-20%)(0603)
- C14, C15: value .1uF -> 22uF; device SparkFun-Capacitors:CAP0805 -> SparkFun-Capacitors:22UF-0805-6.3V-20%
- C16, C17: value .1uF -> 10uF; device SparkFun-Capacitors:CAP0805 -> SparkFun-Capacitors:10UF-0603-6.3V-20%
- C18: value 0.1uF -> 1.0uF; device SparkFun-Capacitors:CAP0805 -> SparkFun-Capacitors:1.0UF-0603-16V-10%
- C19: value 0.1uF -> 10uF; device SparkFun-Capacitors:CAP0805 -> SparkFun-Capacitors:10UF-0603-6.3V-20%
- C2: value 4.7uF -> 0.1uF; device SparkFun-Capacitors:CAP0805 -> SparkFun-Capacitors:0.1UF-25V(+80/-20%)(0603)
- C3: value .22uF -> 0.1uF; device SparkFun-Capacitors:CAP0805 -> SparkFun-Capacitors:0.1UF-25V(+80/-20%)(0603)
- C4: value 0.1uF -> 10nF; device SparkFun-Capacitors:CAP0805 -> SparkFun-Capacitors:10NF/10000PF-50V-10%(0603)
- C5: value 10nF -> 0.1uF; device SparkFun-Capacitors:CAP0805 -> SparkFun-Capacitors:0.1UF-25V(+80/-20%)(0603)
- C6: value 0.1uF -> 15pF; device SparkFun-Capacitors:CAP0805 -> SparkFun-Capacitors:15PF-50V-5%(0603)
- C7: value 2.2nF -> 0.1uF; device SparkFun-Capacitors:CAP0805 -> SparkFun-Capacitors:0.1UF-25V(+80/-20%)(0603)
- C8: value .1uF -> 15pF; device SparkFun-Capacitors:CAP0805 -> SparkFun-Capacitors:15PF-50V-5%(0603)
- J1: value POWER_JACKPTH_LOCK -> 1981584-1; device SparkFun-Connectors:POWER_JACKPTH_LOCK -> audio amplifier example:1981584-1
- JP1, JP2: value (none) -> JUMPER-PAD-3-2OF3_NC_BY_TRACE_SMALL; device SparkFun-Connectors:M03POLAR_LOCK -> SparkFun-Passives:JUMPER-PAD-3-2OF3_NC_BY_TRACE_SMALL
- JP3: device SparkFun-Connectors:M03POLAR_LOCK -> pinhead:PINHD-1X2
- JP4: device SparkFun-Connectors:M03POLAR_LOCK -> pinhead:PINHD-1X3
- JP5: device SparkFun-Connectors:M03POLAR_LOCK -> pinhead:PINHD-1X6
- JP8: device pel_molex:CONN_5-1-53261 -> pinhead:PINHD-1X3
- R1: value 4.7k -> 10K; device SparkFun-Resistors:RESISTOR0805-RES -> SparkFun-Resistors:10KOHM-1/10W-1%(0603)0603
- R10: value 4R -> 330K; device SparkFun-Resistors:RESISTOR2512 -> resistor:R-US_R0603
- R11: value 4R -> 43K; device SparkFun-Resistors:RESISTOR2512 -> resistor:R-US_R0603
- R12: value 3K3 -> 73.2K; device SparkFun-Resistors:RESISTOR0805-RES -> resistor:R-US_R0603
- R13: value 10K -> 22.1; device SparkFun-Resistors:RESISTOR0805-RES -> resistor:R-US_R0603
- R14: value 4.7K -> 100K; device SparkFun-Resistors:RESISTOR0805-RES -> resistor:R-US_R0603
- R15: value 1.33K -> 470k; device SparkFun-Resistors:RESISTOR0805-RES -> resistor:R-US_R0603
- R16: value .1R prec -> 4.7k; device SparkFun-Resistors:RESISTOR0805-RES -> resistor:R-US_R0603
- R17: value 3K3 -> 6.04K; device SparkFun-Resistors:RESISTOR0805-RES -> resistor:R-US_R0603
- R18: value 10K -> 4.7K; device SparkFun-Resistors:RESISTOR0805-RES -> resistor:R-US_R0603
- R19: value 3K3 -> 680; device SparkFun-Resistors:RESISTOR0805-RES -> resistor:R-US_R0603
- R2, R3: device SparkFun-Resistors:RESISTOR0805-RES -> resistor:R-US_R0603
- R20: value 4.7K -> 10K; device SparkFun-Resistors:RESISTOR0805-RES -> resistor:R-US_R0603
- R21: value 10K -> 3.3K; device SparkFun-Resistors:RESISTOR0805-RES -> resistor:R-US_R0603
- R22: value 4.7K -> 1k; device SparkFun-Resistors:RESISTOR0805-RES -> resistor:R-US_R0603
- R23: value 3K3 -> 4; device SparkFun-Resistors:RESISTOR0805-RES -> resistor:R-US_R0603
- R24: value 10K -> 4; device SparkFun-Resistors:RESISTOR0805-RES -> resistor:R-US_R0603
- R25: value 4.7K -> 4.7k; device SparkFun-Resistors:RESISTOR0805-RES -> SparkFun-Resistors:RESISTOR0603
- R26, R27: value 100k -> 4; device SparkFun-Resistors:RESISTOR0805-RES -> resistor:R-US_R0603
- R4: value 316k -> 110K; device SparkFun-Resistors:RESISTOR0805-RES -> SparkFun-Resistors:10KOHM-1/10W-1%(0603)0603
- R5: value 110k -> 316K; device SparkFun-Resistors:RESISTOR0805-RES -> SparkFun-Resistors:10KOHM-1/10W-1%(0603)0603
- R6: value 3K3 -> (none); device SparkFun-Resistors:RESISTOR0805-RES -> SparkFun-Resistors:RESISTOR0603
- R7: value .1R prec -> (none); device SparkFun-Resistors:RESISTOR0805-RES -> SparkFun-Resistors:RESISTOR0603
- R8: value 10K -> 100K; device SparkFun-Resistors:RESISTOR0805-RES -> resistor:R-US_R0603
- R9: value 4.7K -> 40.9K; device SparkFun-Resistors:RESISTOR0805-RES -> resistor:R-US_R0603
- T1, T3, T5: value MOSFET_PCHAN_20A -> NDS352A; device phonesat:MOSFET_PCHAN_20A -> zetex:PMOSSOT23
- T2, T4: value SINGLE_NCHAN_FET -> NDS352A; device phonesat:SINGLE_NCHAN_FET -> zetex:PMOSSOT23
- U1: SPICEPREFIX (none) -> U
- U2: value ARDUINO_PRO_MINI -> LSM9DS1; device SparkFun-Boards:ARDUINO_PRO_MINI -> SparkFun-Sensors:LSM9DS1
- U3: value HMC5883LSMD -> MAX708RESA-T; device SparkFun-Sensors:HMC5883LSMD -> maholli:MAX708RESA-T
- U4: value TEENSY_3.0+4 -> ATSAMD21G-A; device Teensy3.0:TEENSY_3.0+4 -> samd21-temp:ATSAMD21G-A
- U5: value ITG-3200 -> MAX4372TEUK+T; device SparkFun-Sensors:ITG-3200 -> maholli:MAX4372TEUK+T
- U6: value CURRENT_MAX4372 -> MAX4372TEUK+T; device phonesat:CURRENT_MAX4372 -> maholli:MAX4372TEUK+T
- U7: value MURATA_REG_OKL-T3-W12 -> TPS54226PWPRPWP14_2P31X2P46-L; device phonesat:MURATA_REG_OKL-T6-W12 -> maholli:TPS54226PWPRPWP14_2P31X2P46-L
- U8: value CURRENT_MAX4372 -> LTC4121-4.2; device phonesat:CURRENT_MAX4372 -> BrownSpaceEngineering:LTC4121-4.2
- renumbered U$3 to L2
Connections:
- removed net 5V: C11.1, C12.1, R19.2, T7.S@1, T7.S@2, T7.S@3, U1.VCC, U4.VIN, U7.SENSE, U7.VOUT
- removed net BATT_INPUT: J1.PWR, ST1.1, ST2.1, ST3.2
- removed net PGM_RST: S1.2, U2.RST@2
- removed net PGM_VCC: S1.5, U2.VCC
- removed net UART3_RX: JP8.3, U4.7
- removed net UART3_TX: JP8.2, U4.8
- new net !RESET: JP4.2, JP5.3, R1.1, U4.!RESET!
- new net 3.3V_REF: U12.REFP0
- new net A_3.3V: U12.AVDD
- new net DAC_0: JP22.1, U4.PA02(AIN0/DAC)
- new net GPS_1PPS: U11.1PPS, U4.PA03(AIN1/REFA)
- new net I2C_SDOA/G: JP1.2, U2.SDO_A/G
- new net L1_CHG: R8.1, R9.1, U8.RUN
- new net L1_FAULTN: R16.1, U8.~FAULT
- new net L1_PROG: R17.2, U8.PROG
- new net LED_GRN: D2.C, U4.PB08(AIN2/SER4:0/TC4:0)
- new net LION1: C26.1, F1.P$1, R19.2, U8.BAT, U8.BATSNS
- new net N$14: C18.2, U7.VBST
- new net N$15: Q3.G, R40.1, T3.D
- new net N$16: U10.PORT1, X2.1
- new net N$18: C7.1, L1.2, U4.VDDANA
- new net N$20: R47.1, U12.AIN0
- new net N$22: J2.GND, J2.GNDBREAK, JP11.2, JP12.2, JP15.1
- new net N$23: JP20.2, U2.CS_M
- new net N$25: C29.1, R35.2, T2.G
- new net N$26: JP21.2, U2.CS_A/G
- new net N$27: R48.1, U12.AIN1
- new net N$28: C6.2, U4.PA00(XIN32/SER1:0/TC2:0), Y1.2
- new net N$29: C8.1, U4.PA01(XOUT32/SER1:1/TC2:1), Y1.1
- new net N$30: R49.1, U12.AIN2
- new net N$31: IC1.R, R45.2
- new net N$32: C21.2, L4.P$1, U8.SW
- new net N$33: C21.1, U8.BOOST
- new net N$34: C20.1, U8.INTVCC
- new net N$35: R10.1, R11.2, U8.MPPT
- new net N$36: L4.P$2, U8.CHGSNS
- new net N$38: C32.1, R38.2, T5.G
- new net N$41: C27.1, R19.1, U9.VCC
- new net N$45: R22.2, U9.CS
- new net N$46: C25.1, R14.2, U7.VREG5
- new net N$47: Q5.G, R42.1, T5.D
- new net N$48: R51.1, U12.AIN4
- new net N$49: R52.1, U12.AIN5
- new net N$50: R46.1, U12.GPIO0_AIN8
- new net N$51: C24.1, U7.SS
- new net N$52: R12.1, R13.2, U7.VFB
- new net N$53: R53.1, U12.GPIO1_AIN9
- new net N$54: C36.2, U12.REFOUT
- new net N$55: R54.1, U12.GPIO2_AIN10
- new net N$56: R55.1, U12.GPIO3_AIN11
- new net PA04: U4.PA04(AIN4/REFB/SER0:0/TC0:0)
- new net PA12: JP24.1, U4.PA12(I2C/SER2:0+)
- new net PA15: U4.PA15(XOUT/SER2:3+)
- new net PB02: JP28.1, U4.PB02(AIN10/SER5:0)
- new net PB09: JP27.1, U4.PB09(AIN3/SER4:1/TC4:1)
- new net PB10: JP26.1, U4.PB10(SER4:2+)
- new net PB11: JP25.1, U4.PB11(SER4:3+)
- new net PB13: U4.PA13(I2C/SER2:1+)
- new net PGOOD: R14.1, U7.PG
- new net PWR_GND: C14.1, C15.1, C16.2, C17.2, C24.2, C25.2, R13.1, U7.EPAD, U7.GND, U7.PGND1, U7.PGND2
- new net RF_IN: U10.SUM_PORT, U11.RF_IN
- new net SPI_SS2: U12.CS_N
- new net SWCLK: JP5.4, U4.PA30(SWCLK/SER1:2+)
- new net SWDIO: JP5.5, U4.PA31(SWDIO/SER1:3+)
- new net USB_D_N: J1.D-, U4.PA24(SER3:2+)
- new net USB_D_P: J1.D+, U4.PA25(SER3:3+)
- new net USB_ID: J1.ID, JP8.2
- new net VDDCORE3: C10.1, U4.VDDCORE
- new net VSOLAR_IN: C19.1, D1.C, R10.2, R9.2, U8.IN
- new net WDT_!PFO: U3.!PFO, U4.PA20(SER5:2+)
- new net WDT_!RESET: JP4.1, U3.!RESET
- new net WDT_PFI: U3.PFI, U4.PB22(SER5:2+)
- new net WDT_RESET: JP4.3, U3.RESET
- net 3.3V: now also C11.1, C12.1, C14.2, C15.2, C2.1, C22.1, C23.1, C3.1, C9.1, JP1.3, JP2.3, JP20.3, JP21.3, JP3.2, JP5.2, JP8.1, L1.1, L3.P$1, Q1.D, R1.2, R12.2, R15.2, R16.2, R21.1, R23.2, R24.2, R26.2, R27.2, R29.2, R30.2, R32.2, R33.2, R43.2, R44.2, R7.1, U1.VCC, U11.V_BCKP, U12.DVDD, U12.IOVDD, U2.VDD, U2.VDDIO, U4.VDDIN, U4.VDDIO@17, U4.VDDIO@36, U5.VCC, U6.RS-, U7.VO; no longer C14.1, C4.1, C5.1, C8.1, U3.S1, U3.VDD, U3.VDDIO, U4.3.3V, U5.VDD, U5.VLOGIC, U8.VCC
- net ENAB_BURN1: now also R25.2, R35.1, U4.PB23(SER5:3+); no longer R8.1, R9.2, U4.3
- net ENAB_BURN2: now also R28.2, R36.1, U4.PA14(XIN/SER2:2+); no longer R13.1, R14.2, U4.4
- net ENAB_BURN3: now also R31.2, R37.1, U4.PA06(AIN6/SER0:2/TC1:0); no longer R18.1, R20.2, U4.5
- net ENAB_BURN4: now also R34.2, R38.1, U4.PA07(AIN7/SER0:3/TC1:1); no longer R24.1, R25.2, U4.6
- net ENAB_GPS: now also R18.1, R20.2, U4.PA27; no longer R21.1, R22.2, U4.17/A3
- net GND: now also C20.2, C22.2, C23.2, C26.2, C27.2, C28.2, C29.2, C3.2, C30.2, C31.2, C32.2, C33.2, C34.1, C34.2, C36.1, C6.1, J1.GND, J1.S1, JP10.1, JP13.1, JP14.1, JP15.2, JP17.1, JP19.1, JP20.1, JP21.1, JP5.6, JP8.3, JP9.1, R11.1, R17.1, R18.2, R28.1, R31.1, R34.1, R4.1, R8.2, T1.S, T3.S, T5.S, U10.GND, U10.GND@1, U10.GND@10, U10.GND@11, U10.GND@12, U10.GND@13, U10.GND@14, U10.GND@16, U10.GND@17, U10.GND@18, U10.GND@19, U10.GND@2, U10.GND@20, U10.GND@21, U10.GND@22, U10.GND@23, U10.GND@24, U10.GND@25, U10.GND@27, U10.GND@28, U10.GND@29, U10.GND@3, U10.GND@30, U10.GND@31, U10.GND@32, U10.GND@5, U10.GND@6, U10.GND@7, U10.GND@8, U10.GND@9, U11.GND@10, U11.GND@12, U11.GND@13, U11.GND@24, U12.AVSS, U12.AVSS-SW, U12.CLK, U12.DGND, U12.REFCOM, U12.REFN0, U12.START_SYNC, U2.RES, U3.GND, U4.GND@18, U4.GND@35, U4.GND@42, U4.GNDANA, U8.FREQ, U8.NC, U8.NTC, U9.S2, U9.TST, U9.VSS, X1.2, X2.2, X3.2; no longer C14.2, C15.2, C16.2, C17.2, C18.2, C6.2, JP3.1, JP4.1, JP8.1, R1.1, R14.1, R15.2, R20.1, R26.1, R5.1, R9.1, SMA1.2, ST5.2, T10.S, T6.S, T8.S, U2.GND@2, U3.GND@1, U3.GND@2, U4.AGND, U4.GND, U5.AD0, U5.CLKIN, U5.RESV-G, U7.GND1, U7.GND2
- net GPS_PWR: now also Q1.S, U11.VCC; no longer JP8.5, T7.D@1, T7.D@2, T7.D@3, T7.D@4
- net I2C_SCL: now also U11.SCL/NC, U2.SCL/SPC, U4.PA10(AIN18/SER0:2+); no longer U3.SCL, U4.19/A5, U5.SCL
- net I2C_SDA: now also U11.SDA/NC, U2.SDA/SDI/SDO, U4.PA09(I2C/AIN17/SER0:1+); no longer U3.SDA, U4.18/A4, U5.SDA
- net I_BATT: now also U4.PA05(AIN5/SER0:1/TC0:1), U5.OUT; no longer U4.14/A0, U6.OUT
- net I_SOLAR: now also U4.PA08(I2C/AIN16/SER0:0+), U6.OUT; no longer U4.16/A2, U8.OUT
- net N$1: now also D2.A, R43.1; no longer J1.GND, J1.GNDBREAK, ST1.2, ST2.2, ST5.1
- net N$10: now also C28.1, R20.1, T1.G; no longer C16.1, R21.2, T8.G
- net N$11: now also C31.1, R37.2, T4.G; no longer S1.3, U4.23/A9
- net N$12: now also Q1.G, R21.2, T1.D; no longer R19.1, T7.G, T8.D
- net N$13: now also F2.1, J1.VBUS; no longer S1.6, U4.VUSB
- net N$17: now also U10.PORT2, X3.1; no longer C19.1, R26.2, R27.1, U2.A1
- net N$19: now also X1.1; no longer SMA1.1
- net N$2: now also C4.1, U2.CAP; no longer C13.1, R13.2, T4.G
- net N$21: now also JP2.2, U2.SDO_M; no longer C9.1, R8.2, T2.G
- net N$24: now also JP19.3, R44.1; no longer R6.1, T1.G, T2.D
- net N$3: now also C18.1, L3.P$2, U7.SW1, U7.SW2; no longer R12.1, T3.G, T4.D
- net N$37: now also R15.1, U8.~CHRG; no longer C18.1, R4.1, R5.2, U4.15/A1
- net N$39: now also D3.A1, IC1.V-, R45.1; no longer C7.1, U5.CPOUT
- net N$4: now also JP16.1, JP18.2; no longer ST3.1, ST4.2
- net N$40: now also C13.1, R4.2, R5.1, U4.PA11(AIN19/SER0:3+); no longer C6.1, U5.REGOUT
- net N$42: now also C17.1, U7.VCC; no longer C2.1, U3.C1
- net N$43: now also R50.1, U12.AIN3; no longer C3.1, U3.SETP
- net N$44: now also Q4.G, R41.1, T4.D; no longer C3.2, U3.SETC
- net N$5: now also C30.1, R36.2, T3.G; no longer C15.1, R18.2, T6.G
- net N$6: now also C5.1, U2.C1; no longer R17.1, T5.G, T6.D
- net N$7: now also Q2.G, R39.1, T2.D; no longer R15.1, U7.TRIM
- net N$8: now also JP3.1, U3.VCC; no longer C17.1, R24.2, T10.G
- net N$9: now also JP19.2, U11.RSTN; no longer R23.1, T10.D, T9.G
- net N_ENAB_REG: now also U4.PA16(I2C/SER1:0+), U7.EN; no longer R1.2, U2.12, U7.ON/OFF
- net RF_NIRQ: now also U4.PB03(AIN11/SER5:1); no longer U4.2
- net RF_SDN: now also U4.PA19(SER1:3+); no longer U4.9
- net SPI_MISO: now also U12.DIN, U12.DOUT_DRDY_N, U4.PA22(I2C/SER3:0+); no longer U4.12
- net SPI_MOSI: now also U4.PA21(SER5:3+); no longer U4.11
- net SPI_SCK: now also U12.SCLK, U4.PA23(I2C/SER3:0+); no longer U4.13
- net SPI_SS: now also U4.PA28; no longer U4.10
- net UART1_RX: now also U11.TXD, U4.PA18(SER1:2+); no longer U2.TXO, U4.0
- net UART1_TX: now also U11.RXD, U4.PA17(I2C/SER1:1+); no longer U2.RXI, U4.1
- net VBATT: now also C33.1, F1.P$2, F2.2, J2.PWR, JP11.1, JP12.1, JP16.2, JP18.1, R5.2, R6.2, U5.RS+; no longer R10.2, R11.2, R16.1, R27.2, R4.2, R7.2, ST4.1, U2.RAW, U6.RS+, U8.RS-
- net VBURN1: now also JP6.3, Q2.S; no longer JP1.3, T1.D@1, T1.D@2, T1.D@3, T1.D@4
- net VBURN2: now also JP7.3, Q3.S; no longer JP2.3, T3.D@1, T3.D@2, T3.D@3, T3.D@4
- net VBURN3: now also JP10.3, Q4.S; no longer JP3.3, T5.D@1, T5.D@2, T5.D@3, T5.D@4
- net VBURN4: now also JP9.3, Q5.S; no longer JP7.3, T9.D@1, T9.D@2, T9.D@3, T9.D@4
- net VBURN_IN: now also Q2.D, Q3.D, Q4.D, Q5.D, R23.1, R24.1, R26.1, R27.1, R29.1, R30.1, R32.1, R33.1, R39.2, R40.2, R41.2, R42.2; no longer R10.1, R11.1, R12.2, R17.2, R23.2, R6.2, T1.S@1, T1.S@2, T1.S@3, T3.S@1, T3.S@2, T3.S@3, T5.S@1, T5.S@2, T5.S@3, T9.S@1, T9.S@2, T9.S@3
- net VREG_IN: now also C16.1, R6.1, U5.RS-; no longer C10.1, R7.1, U6.RS-
- net VSOLAR: now also D1.A, JP10.2, JP13.2, JP14.2, JP17.2, JP7.2, R7.2, U6.RS+; no longer JP1.2, JP2.2, JP3.2, JP4.2, JP5.2, R16.2, U8.RS+
Other:
- note added: "2s2P Li-Ion Battery Charging Circuit"
- note added: "4"
- note added: "ATSAMD21G18 32-bit ARM Microprocessor VDD Range: 1.62-3.63V"
- note added: "Buck Converter - 3.3V OUT"
- note added: "Burn Wire Control"
- note added: "External WDT"
- note added: "FREQ tied to GND to select 750kHz switching frequency"
- note added: "GPS Module"
- note added: "HopeRF RFM23B module at 3.3V"
- note added: "IMU - LSM9DS1"
- note added: "JTAG"
- note added: "LTC4121 can handle several amps of inrush current upon battery connection"
- note added: "Modifications are currently needed to the module for radiation tolerance"
- note added: "NC tied to ground prevent charge buildup, approved by LT."
- note added: "NTC tied to GND b/c no NTC sensor"
- note added: "Pick Rsense 0.1%"
- note added: "Place L1 near SW pin"
- note added: "Power Connectors: USB, Barrel Plug, Battery"
- note added: "R28 & R29 set Vmp=9V"
- note added: "RF Splitter - 2 Way, 0deg DC-Pass"
- note added: "Run pulled up to ensure charging on startup"
- note added: "Spare IO breakout"
- note added: "To Do: XLab Mez board design Stretch Goals: Ultracap Power Supply Max GFET sensor"
- note added: "Ven threshold is 2.45V. Resistor divider sets RUN high when Solar Panel Voltage is >=6V."
- note added: "Zac Manchester, Max Holliday"
- note removed: "3"
- note removed: "Charging Jack"
- note removed: "Current Limiting Resistors for Burn Wires"
- note removed: "Piksi GPS Connector"
- note removed: "Zac Manchester"
